File: kicad/MaisonEtape1.kicad_sch (KiCad schematic)
At the start: 9 parts, among them J4 AVR-ISP-6, SW1 SW_DIP_x01, SW2 SW_DIP_x01, SW3 SW_DIP_x01, U1 ATmega328-P, U2 ATmega328-P

Commit message: update sur tout le schema
Parts:
- added R15, R16, R17: 10K, symbol Device:R
- added SW4: SW_SPDT, symbol Switch:SW_SPDT
Connections:
- net +5V: now also Lt.20 (AVCC), U1.20 (AVCC), U2.7 (VCC), R15.1, R16.1, R17.1
- net CS: now also SW4.3 (C); no longer Lt.16 (PB2)
- net GND: now also J4.6 (GND)
- net SPI_MISO: now also J4.1 (MISO)
- net SPI_MOSI: now also J4.4 (MOSI)
- net SPI_SCK: now also J4.3 (SCK)
- net at Lt.1 (~{RESET}/PC6): now also J4.5 (~{RST})
- net at J4.1 (MISO): now also U1.17 (PB3); no longer U1.18 (PB4)
- net at J4.4 (MOSI): now also U1.18 (PB4); no longer U1.17 (PB3)
- net at SW1.2, U1.5 (PD3): now also R16.2
- net at SW3.2, U2.2 (PD0): now also R17.2
- net at SW2.2, U1.4 (PD2): now also R15.2
- net at J4.1 (MISO): now also U2.17 (PB3); no longer U2.18 (PB4)
- net at J4.4 (MOSI): now also U2.18 (PB4); no longer U2.17 (PB3)
- new net: Lt.16 (PB2), SW4.2 (B)
Other:
- sheet Photon renamed ESP32
- note added: "Fenetre1"
- note added: "Fenetre2"
- note removed: "F1"
- note removed: "F2"
- moved on the sheet: J4, Lt, SW1, SW2, SW3, U1, U2

Commit message: lfg
Parts:
- removed SW4: SW_SPDT, symbol Switch:SW_SPDT
- added R20, R25, R27: 220R, symbol Device:R
- added R21, R24, R26: 1.5k, symbol Device:R
- added R22, R23: 80k, symbol Device:R
- added R28: 10K, symbol Device:R
- R17: value 10K -> 80k
Connections:
- net +5V: now also R15.2, R28.1; no longer R15.1, R17.1
- net GND: now also R21.1, R24.1, R26.1
- net CS1: now reaches Lt.4 (PD2)
- net CS2: now reaches Lt.5 (PD3)
- net CS3: now reaches Lt.6 (PD4)
- net at R16.2, SW1.2: now also R20.2; no longer U1.5 (PD3)
- net at U2.13 (PD7): now also R17.1
- net at U1.12 (PD6): now also R23.1
- net at U1.13 (PD7): now also R22.1
- new net: R27.2, R28.2, SW3.2
- new net: R20.1, R21.2, R22.2
- new net: R15.1, R25.2, SW2.2
- new net: R23.2, R24.2, R25.1
- new net: R17.2, R26.2, R27.1
- now unconnected: U1.4 (PD2), U2.2 (PD0)
Other:
- note removed: "Porte"
- moved on the sheet: J4, Lt, R15, R16, SW1, SW2
