File: kicad/MaisonEtape1.kicad_sch (KiCad schematic)
At the start: 25 parts, among them J14 Conn_01x08_Socket, J4 AVR-ISP-6, J5 Conn_01x08_Socket, U1 ATmega8A-A, U2 ATmega8A-A

Commit message: update kicad
Parts:
- added R29, R30, R31: 220, Resistor_SMD:R_0805_2012Metric_Pad1.20x1.40mm_HandSolder, symbol Device:R
- added Window_1, Window_2, door_1: LED, LED_SMD:LED_0805_2012Metric, symbol Device:LED
- J14, J5: footprint (none) -> Connector_PinHeader_2.54mm:PinHeader_1x08_P2.54mm_Vertical
- renumbered Door to Door1, LT to LT1
Connections:
- net U1_GND: now also Window_1.1 (K), Window_2.1 (K)
- net U2_GND: now also door_1.1 (K)
- net at U2.12 (PB0): now also R31.1
- net at U1.12 (PB0): now also R29.1
- net at U1.13 (PB1): now also R30.1
- new net: R31.2, door_1.2 (A)
- new net: R29.2, Window_1.2 (A)
- new net: R30.2, Window_2.2 (A)

Commit message: update friday pcb
Parts:
- J4: footprint Connector_IDC:IDC-Header_2x03_P2.54mm_Vertical -> JPLibrary:SPI_prog
- J_U2: footprint Connector_PinHeader_2.54mm:PinHeader_1x04_P2.54mm_Vertical -> Connector_PinSocket_2.54mm:PinSocket_1x04_P2.54mm_Vertical
- renumbered J5 to J13
Changed lines of the file:
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@@
       (effects (font (size 1.27 1.27)) (justify right))
     )
-    (property "Footprint" "Connector_IDC:IDC-Header_2x03_P2.54mm_Vertical" (at 87.63 95.25 90)
+    (property "Footprint" "JPLibrary:SPI_prog" (at 87.63 95.25 90)
       (effects (font (size 1.27 1.27)) hide)
     )
@@
       (effects (font (size 1.27 1.27)) (justify left))
     )
-    (property "Footprint" "Connector_PinHeader_2.54mm:PinHeader_1x04_P2.54mm_Vertical" (at 152.4 156.21 0)
+    (property "Footprint" "Connector_PinSocket_2.54mm:PinSocket_1x04_P2.54mm_Vertical" (at 152.4 156.21 0)
       (effects (font (size 1.27 1.27)) hide)
     )
@@
       (effects (font (size 1.27 1.27)) (justify right))
     )
-    (property "Footprint" "Connector_IDC:IDC-Header_2x03_P2.54mm_Vertical" (at 270.51 92.71 90)
+    (property "Footprint" "JPLibrary:SPI_prog" (at 270.51 92.71 90)
       (effects (font (size 1.27 1.27)) hide)
     )
@@
   (symbol (lib_id "Connector:Conn_01x08_Socket") (at 261.62 127 0) (unit 1)
     (in_bom yes) (on_board yes) (dnp no) (fields_autoplaced)
-    (property "Reference" "J5" (at 262.89 128.27 0)
+    (property "Reference" "J13" (at 262.89 128.27 0)
       (effects (font (size 1.27 1.27)) (justify left))
     )
@@
       (project "MaisonEtape1"
         (path "/ed06f8de-d1bb-4b1a-bfe3-5df11d3a9162"
-          (reference "J5") (unit 1)
+          (reference "J13") (unit 1)
         )
       )
@@
       (effects (font (size 1.27 1.27)) (justify right))
     )
-    (property "Footprint" "Connector_IDC:IDC-Header_2x03_P2.54mm_Vertical" (at 171.45 95.25 90)
-      (effects (font (size 1.27 1.27)) hide)
-    )
+    (property "Footprint" "JPLibrary:SPI_prog" (at 171.45 95.25 90)
+      (effects (font (size 1.27 1.27)) hide)
+    )

Commit message: kicad update, finalizing
Parts:
- added C5 (x3), C6 (x3): 16pF, Capacitor_SMD:C_0805_2012Metric_Pad1.18x1.45mm_HandSolder, symbol Device:C
- added LT_XT1: Conn_01x09, JP_Library:XT_9, symbol Connector_Generic:Conn_01x09
- added U1_XT1: Conn_01x09, JP_Library:XT_13, symbol Connector_Generic:Conn_01x13
- added U2_XT1: Conn_01x09, JP_Library:XT_15, symbol Connector_Generic:Conn_01x15
- added Y3 (x3): Crystal, JP_Library:Crystal 49SS-SMD, symbol Device:Crystal
- Door1, Window1, Window2: footprint Connector_PinHeader_2.54mm:PinHeader_1x02_P2.54mm_Vertical -> Connector_PinSocket_2.54mm:PinSocket_1x02_P2.54mm_Vertical
- J_U2: footprint Connector_PinSocket_2.54mm:PinSocket_1x04_P2.54mm_Vertical -> Connector_PinHeader_2.54mm:PinHeader_1x04_P2.54mm_Vertical
Connections:
- net +5V is gone; now on net LT_VCC: J4.2 (VCC)
- net GND is gone; now on net LT_GND: J4.6 (GND)
- net LT_GND: now also J13.2 (Pin_2), LT1.21 (AGND), C5.2, C6.2; no longer J13.8 (Pin_8)
- net U1_GND: now also U1.21 (AGND), C5.2, C6.2
- net U2_GND: now also U2.21 (AGND), C5.2, C6.2
- net U2_PD3: now reaches U2.1 (PD3)
- net U2_PD3: now also U2_XT1.12 (Pin_12)
- net U2_PD6: now reaches U2.10 (PD6)
- net U2_PD6: now also U2_XT1.15 (Pin_15)
- net U2_PB1: now reaches U2.13 (PB1)
- net U2_PB1: now also U2_XT1.3 (Pin_3)
- net U2_PB2: now reaches U2.14 (PB2)
- net U2_PB2: now also U2_XT1.4 (Pin_4)
- net U2_ADC6: now reaches U2.19 (ADC6)
- net U2_ADC6: now also U2_XT1.1 (Pin_1)
- net U2_PD4: now reaches U2.2 (PD4)
- net U2_PD4: now also U2_XT1.13 (Pin_13)
- net U2_ADC7: now reaches U2.22 (ADC7)
- net U2_ADC7: now also U2_XT1.2 (Pin_2)
- net U2_PC0: now reaches U2.23 (PC0)
- net U2_PC0: now also U2_XT1.5 (Pin_5)
- net U2_PC1: now reaches U2.24 (PC1)
- net U2_PC1: now also U2_XT1.6 (Pin_6)
- net U2_PC2: now reaches U2.25 (PC2)
- net U2_PC2: now also U2_XT1.7 (Pin_7)
- net U2_PC3: now reaches U2.26 (PC3)
- net U2_PC3: now also U2_XT1.8 (Pin_8)
- net U2_PD0: now reaches U2.30 (PD0)
- net U2_PD0: now also U2_XT1.9 (Pin_9)
- net U2_PD1: now reaches U2.31 (PD1)
- net U2_PD1: now also U2_XT1.10 (Pin_10)
- net U2_PD2: now reaches U2.32 (PD2)
- net U2_PD2: now also U2_XT1.11 (Pin_11)
- net U2_PB6: now reaches U2.7 (PB6/XTAL1)
- net U2_PB6: now also C5.1, Y3.2
- net U2_PB7: now reaches U2.8 (PB7/XTAL2)
- net U2_PB7: now also C6.1, Y3.1
- net U2_PD5: now reaches U2.9 (PD5)
- net U2_PD5: now also U2_XT1.14 (Pin_14)
- net LT_PB0: now reaches LT1.12 (PB0)
- net LT_PB0: now also LT_XT1.3 (Pin_3)
- net LT_PB1: now reaches LT1.13 (PB1)
- net LT_PB1: now also LT_XT1.4 (Pin_4)
- net LT_PB2: now reaches LT1.14 (PB2)
- net LT_PB2: now also LT_XT1.5 (Pin_5)
- net LT_ADC6: now reaches LT1.19 (ADC6)
- net LT_ADC6: now also LT_XT1.1 (Pin_1)
- net LT_ADC7: now reaches LT1.22 (ADC7)
- net LT_ADC7: now also LT_XT1.2 (Pin_2)
- net LT_PC0: now reaches LT1.23 (PC0)
- net LT_PC0: now also LT_XT1.6 (Pin_6)
- net LT_PC1: now reaches LT1.24 (PC1)
- net LT_PC1: now also LT_XT1.7 (Pin_7)
- net LT_PC2: now reaches LT1.25 (PC2)
- net LT_PC2: now also LT_XT1.8 (Pin_8)
- net LT_PC3: now reaches LT1.26 (PC3)
- net LT_PC3: now also LT_XT1.9 (Pin_9)
- net LT_PB6: now reaches LT1.7 (PB6/XTAL1)
- net LT_PB6: now also C5.1, Y3.2
- net LT_PB7: now reaches LT1.8 (PB7/XTAL2)
- net LT_PB7: now also C6.1, Y3.1
- net D3: now reaches U1.1 (PD3)
- net D3: now also U1_XT1.11 (Pin_11)
- net B2: now reaches U1.14 (PB2)
- net B2: now also U1_XT1.3 (Pin_3)
- net A6: now reaches U1.19 (ADC6)
- net A6: now also U1_XT1.1 (Pin_1)
- net D4: now reaches U1.2 (PD4)
- net D4: now also U1_XT1.12 (Pin_12)
- net A7: now reaches U1.22 (ADC7)
- net A7: now also U1_XT1.2 (Pin_2)
- net C0: now reaches U1.23 (PC0)
- net C0: now also U1_XT1.4 (Pin_4)
- net C1: now reaches U1.24 (PC1)
- net C1: now also U1_XT1.5 (Pin_5)
- net C2: now reaches U1.25 (PC2)
- net C2: now also U1_XT1.6 (Pin_6)
- net C3: now reaches U1.26 (PC3)
- net C3: now also U1_XT1.7 (Pin_7)
- net D0: now reaches U1.30 (PD0)
- net D0: now also U1_XT1.8 (Pin_8)
- net D1: now reaches U1.31 (PD1)
- net D1: now also U1_XT1.9 (Pin_9)
- net D2: now reaches U1.32 (PD2)
- net D2: now also U1_XT1.10 (Pin_10)
- net U1_PB6: now reaches U1.7 (PB6/XTAL1)
- net U1_PB6: now also C5.1, Y3.2
- net U1_PB7: now reaches U1.8 (PB7/XTAL2)
- net U1_PB7: now also C6.1, Y3.1
- net D5: now reaches U1.9 (PD5)
- net D5: now also U1_XT1.13 (Pin_13)
- net CS1 renamed LT_CS1
- net LT_CS1: now also J13.3 (Pin_3); no longer J13.2 (Pin_2)
- net CS2 renamed LT_CS2
- net LT_CS2: now also J13.4 (Pin_4); no longer J13.3 (Pin_3)
- net CS3 renamed LT_CS3
- net LT_CS3: now also J13.5 (Pin_5); no longer J13.4 (Pin_4)
- net CS4 renamed LT_CS4
- net LT_CS4: now also J13.6 (Pin_6); no longer J13.5 (Pin_5)
- net CS5 renamed LT_CS5
- net LT_CS5: now also J13.7 (Pin_7); no longer J13.6 (Pin_6)
- net CS6 renamed LT_CS6
- net LT_CS6: now also J13.8 (Pin_8); no longer J13.7 (Pin_7)
Other:
- moved on the sheet: Door1, J13, J14, J4, J_U1, J_U2, LT1, R15, R16, R17, R20, R21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

Commit message: update U6
Parts:
- added J_U3: Conn_01x04_Socket, Connector_PinHeader_2.54mm:PinHeader_1x04_P2.54mm_Vertical, symbol Connector:Conn_01x04_Socket
- added U9: DS1621, Package_DIP:DIP-8_W7.62mm, symbol Sensor_Temperature:DS1621
Connections:
- new net U6_GND: J_U3.2 (Pin_2), U9.4 (GND), U9.5 (A2), U9.6 (A1), U9.7 (A0)
- new net U6_VCC: J_U3.1 (Pin_1), U9.8 (V_{DD})
- new net U6_i2c_SCL: J_U3.3 (Pin_3), U9.2 (SCL)
- new net U6_i2c_SDA: J_U3.4 (Pin_4), U9.1 (SDA)
- no-connect marks 0 -> 1
Changed lines of the file:
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@@
   (junction (at 41.91 148.59) (diameter 0) (color 0 0 0 0)
   )
+  (no_connect (at 59.69 27.94))
   (wire (pts (xy 162.56 140.97) (xy 162.56 137.16))
     (stroke (width 0) (type default))
@@
     (stroke (width 0) (type default))
   )
+  (wire (pts (xy 46.99 38.1) (xy 46.99 40.64))
+    (stroke (width 0) (type default))
+  )
   (wire (pts (xy 30.48 57.15) (xy 33.02 57.15))
     (stroke (width 0) (type default))
@@
   )
   (wire (pts (xy 213.36 147.32) (xy 213.36 151.13))
+    (stroke (width 0) (type default))
+  )
+  (wire (pts (xy 46.99 15.24) (xy 46.99 17.78))
     (stroke (width 0) (type default))
   )
@@
     (effects (font (size 4 4)) (justify left bottom))
   )
+  (label "U6" (at 17.78 20.32 0) (fields_autoplaced)
+    (effects (font (size 4 4)) (justify left bottom))
+  )
   (label "i2C SECTION" (at 106.68 43.18 0) (fields_autoplaced)
     (effects (font (size 6 6)) (justify left bottom))
@@
     )
   )
+  (global_label "U6_GND" (shape input) (at 46.99 40.64 180) (fields_autoplaced)
+    (effects (font (size 1.27 1.27)) (justify right))
+    (property "Intersheetrefs" "${INTERSHEET_REFS}" (at 36.7061 40.64 0)
+      (effects (font (size 1.27 1.27)) (justify right) hide)
+    )
+  )
   (global_label "U1_i2c_SCL" (shape input) (at 34.29 160.02 180) (fields_autoplaced)
     (effects (font (size 1.27 1.27)) (justify right))
@@
     )
   )
+  (global_label "U6_GND" (shape input) (at 34.29 30.48 180) (fields_autoplaced)
+    (effects (font (size 1.27 1.27)) (justify right))
+    (property "Intersheetrefs" "${INTERSHEET_REFS}" (at 24.0061 30.48 0)
+      (effects (font (size 1.27 1.27)) (justify right) hide)
+    )
+  )
   (global_label "LT_UART_RX" (shape input) (at 229.87 116.84 0) (fields_autoplaced)
     (effects (font (size 1.27 1.27)) (justify left))
@@
     )
   )
+  (global_label "U6_GND" (shape input) (at 34.29 27.94 180) (fields_autoplaced)
+    (effects (font (size 1.27 1.27)) (justify right))
+    (property "Intersheetrefs" "${INTERSHEET_REFS}" (at 24.0061 27.94 0)
+      (effects (font (size 1.27 1.27)) (justify right) hide)
+    )
+  )
+  (global_label "U6_VCC" (shape input) (at 46.99 15.24 180) (fields_autoplaced)
+    (effects (font (size 1.27 1.27)) (justify right))
+    (property "Intersheetrefs" "${INTERSHEET_REFS}" (at 36.948 15.24 0)
+      (effects (font (size 1.27 1.27)) (justify right) hide)
+    )
+  )
   (global_label "U1_PB7" (shape input) (at 26.67 93.98 180) (fields_autoplaced)
     (effects (font (size 1.27 1.27)) (justify right))
@@
     )
   )
+  (global_label "U6_i2c_SDA" (shape input) (at 91.44 29.21 180) (fields_autoplaced)
+    (effects (font (size 1.27 1.27)) (justify right))
+    (property "Intersheetrefs" "${INTERSHEET_REFS}" (at 77.588 29.21 0)
+      (effects (font (size 1.27 1.27)) (justify right) hide)
+    )
+  )
   (global_label "U1_GND" (shape input) (at 64.77 157.48 0) (fields_autoplaced)
     (effects (font (size 1.27 1.27)) (justify left))
@@
     )
   )
+  (global_label "U6_GND" (shape input) (at 91.44 24.13 180) (fields_autoplaced)
+    (effects (font (size 1.27 1.27)) (justify right))
+    (property "Intersheetrefs" "${INTERSHEET_REFS}" (at 81.1561 24.13 0)
+      (effects (font (size 1.27 1.27)) (justify right) hide)
+    )
+  )
   (global_label "LT_UART_TX" (shape input) (at 229.87 119.38 0) (fields_autoplaced)
     (effects (font (size 1.27 1.27)) (justify left))
@@
     )
   )
+  (global_label "U6_GND" (shape input) (at 34.29 33.02 180) (fields_autoplaced)
+    (effects (font (size 1.27 1.27)) (justify right))
+    (property "Intersheetrefs" "${INTERSHEET_REFS}" (at 24.0061 33.02 0)
+      (effects (font (size 1.27 1.27)) (justify right) hide)
+    )
+  )
   (global_label "LT_CS2" (shape input) (at 255.27 127 180) (fields_autoplaced)
     (effects (font (size 1.27 1.27)) (justify right))
@@
     )
   )
+  (global_label "U6_VCC" (shape input) (at 91.44 21.59 180) (fields_autoplaced)
+    (effects (font (size 1.27 1.27)) (justify right))
+    (property "Intersheetrefs" "${INTERSHEET_REFS}" (at 81.398 21.59 0)
+      (effects (font (size 1.27 1.27)) (justify right) hide)
+    )
+  )
   (global_label "D4" (shape input) (at 57.15 129.54 0) (fields_autoplaced)
     (effects (font (size 1.27 1.27)) (justify left))
@@
     )
   )
+  (global_label "U6_i2c_SCL" (shape input) (at 91.44 26.67 180) (fields_autoplaced)
+    (effects (font (size 1.27 1.27)) (justify right))
+    (property "Intersheetrefs" "${INTERSHEET_REFS}" (at 77.6485 26.67 0)
+      (effects (font (size 1.27 1.27)) (justify right) hide)
+    )
+  )
   (global_label "U1_RESET" (shape input) (at 25.4 83.82 180) (fields_autoplaced)
     (effects (font (size 1.27 1.27)) (justify right))
@@
     )
   )
+  (global_label "U6_i2c_SCL" (shape input) (at 34.29 25.4 180) (fields_autoplaced)
+    (effects (font (size 1.27 1.27)) (justify right))
+    (property "Intersheetrefs" "${INTERSHEET_REFS}" (at 20.4985 25.4 0)
+      (effects (font (size 1.27 1.27)) (justify right) hide)
+    )
+  )
   (global_label "LT_CS1" (shape input) (at 229.87 121.92 0) (fields_autoplaced)
     (effects (font (size 1.27 1.27)) (justify left))
@@
     (property "Intersheetrefs" "${INTERSHEET_REFS}" (at 223.0996 151.13 0)
       (effects (font (size 1.27 1.27)) (justify left) hide)
+    )
+  )
+  (global_label "U6_i2c_SDA" (shape input) (at 34.29 22.86 180) (fields_autoplaced)
+    (effects (font (size 1.27 1.27)) (justify right))
+    (property "Intersheetrefs" "${INTERSHEET_REFS}" (at 20.438 22.86 0)
+      (effects (font (size 1.27 1.27)) (justify right) hide)
     )
   )
@@
     )
   )
+  (symbol (lib_id "Connector:Conn_01x04_Socket") (at 96.52 24.13 0) (unit 1)
+    (in_bom yes) (on_board yes) (dnp no) (fields_autoplaced)
+    (property "Reference" "J_U3" (at 97.79 24.13 0)
+      (effects (font (size 1.27 1.27)) (justify left))
+    )
+    (property "Value" "Conn_01x04_Socket" (at 97.79 26.67 0)
+      (effects (font (size 1.27 1.27)) (justify left) hide)
+    )
+    (property "Footprint" "Connector_PinHeader_2.54mm:PinHeader_1x04_P2.54mm_Vertical" (at 96.52 24.13 0)
+      (effects (font (size 1.27 1.27)) hide)
+    )
+    (property "Datasheet" "~" (at 96.52 24.13 0)
+      (effects (font (size 1.27 1.27)) hide)
+    )
+    (pin "1")
+    (pin "2")
+    (pin "3")
+    (pin "4")
+    (instances
+      (project "MaisonEtape1"
+        (path "/ed06f8de-d1bb-4b1a-bfe3-5df11d3a9162"
+          (reference "J_U3") (unit 1)
+        )
+      )
+    )
+  )
   (symbol (lib_id "Connector_Generic:Conn_01x15") (at 143.51 170.18 90) (unit 1)
     (in_bom yes) (on_board yes) (dnp no) (fields_autoplaced)
@@
         )
       )
+    )
+  )
+  (symbol (lib_id "Sensor_Temperature:DS1621") (at 46.99 27.94 0) (unit 1)
+    (in_bom yes) (on_board yes) (dnp no) (fields_autoplaced)
+    (property "Reference" "U9" (at 62.23 24.0539 0)
+      (effects (font (size 1.27 1.27)))
+    )
+    (property "Value" "DS1621" (at 62.23 26.5939 0)
+      (effects (font (size 1.27 1.27)))
+    )
+    (property "Footprint" "Package_DIP:DIP-8_W7.62mm" (at 29.21 36.83 0)
+      (effects (font (size 1.27 1.27)) hide)
+    )
+    (property "Datasheet" "https://datasheets.maximintegrated.com/en/ds/DS1621.pdf" (at 43.18 21.59 0)
+      (effects (font (size 1.27 1.27)) hide)
+    )
+    (pin "1")
+    (pin "2")
+    (pin "3")
+    (pin "4")
+    (pin "5")
+    (pin "6")
+    (pin "7")
+    (pin "8")
+    (instances
+      (project "MaisonEtape1"
+        (path "/ed06f8de-d1bb-4b1a-bfe3-5df11d3a9162"
+          (reference "U9") (unit 1)
+        )
+      )
