File: kicad/_autosave-MaisonEtape1.kicad_sch (KiCad schematic)
At the start: 25 parts, among them J14 Conn_01x08_Socket, J4 AVR-ISP-6, J5 Conn_01x08_Socket, U1 ATmega8A-A, U2 ATmega8A-A

Commit message: 13-10
Parts:
- renumbered Door to Door1, LT to LT1
Changed lines of the file:
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@@
         )
         (path "/ed06f8de-d1bb-4b1a-bfe3-5df11d3a9162"
-          (reference "Jmaster") (unit 1)
+          (reference "Jmaster1") (unit 1)
         )
       )
@@
   (symbol (lib_id "MCU_Microchip_ATmega:ATmega8A-A") (at 212.09 109.22 0) (unit 1)
     (in_bom yes) (on_board yes) (dnp no)
-    (property "Reference" "LT" (at 215.3159 68.58 0)
+    (property "Reference" "LT1" (at 215.3159 68.58 0)
       (effects (font (size 1.27 1.27)) (justify left))
     )
@@
       (project "MaisonEtape1"
         (path "/ed06f8de-d1bb-4b1a-bfe3-5df11d3a9162"
-          (reference "LT") (unit 1)
+          (reference "LT1") (unit 1)
         )
       )
@@
   (symbol (lib_id "Connector:Conn_01x02_Socket") (at 179.07 132.08 90) (unit 1)
     (in_bom yes) (on_board yes) (dnp no)
-    (property "Reference" "Door" (at 171.45 139.7 90)
+    (property "Reference" "Door1" (at 171.45 139.7 90)
       (effects (font (size 1.27 1.27)) (justify right))
     )
@@
       (project "MaisonEtape1"
         (path "/ed06f8de-d1bb-4b1a-bfe3-5df11d3a9162"
-          (reference "Door") (unit 1)
-        )
-      )
+          (reference "Door1") (unit 1)
+        )
+      )
