File: kicad/MaisonEtape1.kicad_pcb (KiCad board)
At the start: 2 copper layers, 100 x 100 mm, 32 parts, among them J1 AVR-ISP-6, J13 AVR-ISP-6, J2 AVR-ISP-6, J3 AVR-ISP-6, J4 AVR-ISP-6, U1 ATmega8A-A, U2 ATmega8A-A, U3 ATmega8A-A, U4 ATmega8A-A, U5 ATmega8A-A

Commit message: update kicad
Parts:
- added J11: Conn_01x02_Socket, Connector_PinSocket_2.54mm:PinSocket_1x02_P2.54mm_Vertical, F.Cu at (136.1, 98.3)
- added J12: Conn_01x02_Socket, Connector_PinSocket_2.54mm:PinSocket_1x02_P2.54mm_Vertical, F.Cu at (78.7, 88.6)
- added J14: Conn_01x08_Socket, Connector_PinHeader_2.54mm:PinHeader_1x08_P2.54mm_Vertical, F.Cu at (133.8, 45.4)
- added J5: Conn_01x08_Socket, Connector_PinHeader_2.54mm:PinHeader_1x08_P2.54mm_Vertical, F.Cu at (133.8, 49.8)
- added Q1: NMOS, Package_TO_SOT_THT:TO-220-3_Vertical, F.Cu at (134.1, 105.4)
- added Q2: NMOS, Package_TO_SOT_THT:TO-220-3_Vertical, F.Cu at (68.1, 84.4)
- added R1: 200R, Resistor_SMD:R_0805_2012Metric_Pad1.20x1.40mm_HandSolder, F.Cu at (78.8, 76.0)
- added R18: 1K, Resistor_SMD:R_0805_2012Metric_Pad1.20x1.40mm_HandSolder, F.Cu at (78.8, 81.9)
- added R19: 200R, Resistor_SMD:R_0805_2012Metric_Pad1.20x1.40mm_HandSolder, F.Cu at (78.8, 84.8)
- added R2: 1K, Resistor_SMD:R_0805_2012Metric_Pad1.20x1.40mm_HandSolder, F.Cu at (78.8, 78.9)
- added R29: 220, Resistor_SMD:R_0805_2012Metric_Pad1.20x1.40mm_HandSolder, B.Cu at (142.0, 63.3)
- added R30: 220, Resistor_SMD:R_0805_2012Metric_Pad1.20x1.40mm_HandSolder, B.Cu at (142.0, 70.4)
- added R31: 220, Resistor_SMD:R_0805_2012Metric_Pad1.20x1.40mm_HandSolder, F.Cu at (140.4, 83.3)
- added SW5: SW_SPDT, Button_Switch_THT:SW_E-Switch_EG1271_SPDT, F.Cu at (67.6, 88.0)
- added Window_1: LED, LED_SMD:LED_0805_2012Metric, F.Cu at (141.9, 70.4)
- added Window_2: LED, LED_SMD:LED_0805_2012Metric, F.Cu at (141.9, 63.3)
- added door_1: LED, LED_SMD:LED_0805_2012Metric, F.Cu at (140.8, 79.7)
- J_SPI_3, J_SPI_4: footprint Connector:NS-Tech_Grove_1x04_P2mm_Vertical -> Connector_PinHeader_2.54mm:PinHeader_1x04_P2.54mm_Vertical
- moved J_SPI_3 108.1 mm to (146.3, 98.3)
- moved Door1 91.8 mm to (137.0, 79.7), turned to -90 degrees
- moved R17 90.1 mm to (132.4, 87.0), turned to 90 degrees
- moved R26 84.8 mm to (135.3, 87.0), turned to 90 degrees
- moved J3 71.1 mm to (107.2, 103.0), turned to 90 degrees
- moved J2 69.5 mm to (107.1, 84.6), turned to 90 degrees
- moved J13 68.2 mm to (21.0, 129.5)
- moved R28 63.3 mm to (141.2, 87.0), turned to 90 degrees
- moved R27 62.1 mm to (138.3, 87.0), turned to 90 degrees
- moved J_SPI_5 54.7 mm to (67.3, 148.9)
- moved U3 54.1 mm to (125.3, 101.9)
- moved J_U2 37.7 mm to (145.9, 79.7)
- moved U2 29.8 mm to (125.1, 83.5)
- moved Window1 25.3 mm to (136.9, 63.0)
- moved LT1 20.4 mm to (125.3, 47.5)
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- renumbered LT to LT1
Connections:
- U1 pad 12: unconnected-(U1-PB0-Pad12) -> Net-(U1-PB0)
- U1 pad 13: unconnected-(U1-PB1-Pad13) -> Net-(U1-PB1)
- U2 pad 12: unconnected-(U2-PB0-Pad12) -> Net-(U2-PB0)
- U3 pad 18: +5V -> U3_VCC
- U3 pad 3: GND -> U3_GND
- U3 pad 4: +5V -> U3_VCC
- U3 pad 5: GND -> U3_GND
- U3 pad 6: +5V -> U3_VCC
- U4 pad 18: +5V -> U4_VCC
- U4 pad 3: GND -> U4_GND
- U4 pad 4: +5V -> U4_VCC
- U4 pad 5: GND -> U4_GND
- U4 pad 6: +5V -> U4_VCC
- U5 pad 18: +5V -> U5_VCC
- U5 pad 21: GND -> U5_GND
- U5 pad 4: +5V -> U5_VCC
- U5 pad 6: +5V -> U5_VCC
Routing:
- net U1_VCC: track 59.2 -> 0.00 mm, vias 2 -> 0
- net U1_i2c_SCL: track 32.7 -> 0.00 mm, vias 2 -> 0
- net Net-(J1-MOSI): track 32.0 -> 0.00 mm, vias 1 -> 0
- net U1_i2c_SDA: track 25.0 -> 0.00 mm, vias 2 -> 0
- net Net-(J1-MISO): track 21.3 -> 0.00 mm
- net U1_RESET: track 20.8 -> 0.00 mm
- net Net-(U1-PD7): track 19.3 -> 0.00 mm, vias 1 -> 0
- net Net-(Window1-Pin_1): track 17.1 -> 0.00 mm, vias 1 -> 0
- net U1_GND: track 15.9 -> 0.00 mm, vias 2 -> 0
- net Net-(R23-Pad2): track 15.2 -> 0.00 mm
- net Net-(Window2-Pin_1): track 13.7 -> 0.00 mm
- net Net-(J1-SCK): track 13.2 -> 0.00 mm
- net Net-(R20-Pad1): track 5.08 -> 0.00 mm
- net Net-(U1-PD6): track 4.74 -> 0.00 mm, vias 1 -> 0
Other:
- outline, holes or cut-outs redrawn
- copper layers 2 -> 4
- board text added: "+"
- board text added: "-"
- board text added: "CS1"
- board text added: "CS2"
- board text added: "CS3"
- board text added: "CS4"
- board text added: "CS5"
- board text added: "CS6"
- board text added: "MISO"
- board text added: "MOSI"
- board text added: "RX"
- board text added: "SCK"
- board text added: "TX"

Commit message: kicadery
Parts:
- J_U2: footprint Connector_PinHeader_2.54mm:PinHeader_1x04_P2.54mm_Vertical -> Connector_PinSocket_2.54mm:PinSocket_1x04_P2.54mm_Vertical
- moved J_SPI_4 101.9 mm to (146.1, 114.3)
- moved U4 78.1 mm to (125.3, 119.1)
- moved SW5 24.9 mm to (82.6, 107.8)
- moved J12 12.2 mm to (79.2, 100.8)
Other:
- outline, holes or cut-outs redrawn
Changed lines of the file:
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@@
     (property "ki_keywords" "connector")
     (attr through_hole)
-    (fp_text reference "J_U1" (at 0 -2.33) (layer "F.SilkS")
+    (fp_text reference "J_U1" (at 0 -2.33) (layer "F.SilkS") hide
         (effects (font (size 1 1) (thickness 0.15)))
     )
@@
   )
   (footprint "Connector_PinHeader_2.54mm:PinHeader_1x04_P2.54mm_Vertical" (layer "F.Cu")
-    (at 45.8 96.055)
+    (at 146.05 114.3)
     (descr "Through hole straight pin header, 1x04, 2.54mm pitch, single row")
     (tags "Through hole pin header THT 1x04 2.54mm single row")
@@
     (property "ki_keywords" "connector")
     (attr through_hole)
-    (fp_text reference "J_SPI_4" (at 0 -2.33) (layer "F.SilkS")
+    (fp_text reference "J_SPI_4" (at 0 -2.33) (layer "F.SilkS") hide
         (effects (font (size 1 1) (thickness 0.15)))
     )
-    (fp_text value "SPI_SOCKET" (at 0 9.95) (layer "F.Fab")
+    (fp_text value "SPI_SOCKET" (at 0 9.95) (layer "F.Fab") hide
         (effects (font (size 1 1) (thickness 0.15)))
     )
@@
   )
   (footprint "Button_Switch_THT:SW_E-Switch_EG1271_SPDT" (layer "F.Cu")
-    (at 67.575 88.016)
+    (at 82.63 107.798)
     (descr "E-Switch sub miniature slide switch, EG series, SPDT, https://www.e-switch.com/wp-content/uploads/2022/06/EG.pdf")
     (tags "switch SPDT")
@@
   )
   (footprint "Package_QFP:TQFP-32_7x7mm_P0.8mm" (layer "F.Cu")
-    (at 49.09 136.15)
+    (at 125.29 119.132)
     (descr "32-Lead Plastic Thin Quad Flatpack (PT) - 7x7x1.0 mm Body, 2.00 mm [TQFP] (see Microchip Packaging Specification 00000049BS.pdf)")
     (tags "QFP 0.8")
@@
     (property "ki_keywords" "AVR 8bit Microcontroller MegaAVR")
     (attr smd)
-    (fp_text reference "U4" (at 0 -6.05) (layer "F.SilkS")
+    (fp_text reference "U4" (at -4.386 -4.324) (layer "F.SilkS")
         (effects (font (size 1 1) (thickness 0.15)))
     )
@@
   )
   (footprint "Connector_PinSocket_2.54mm:PinSocket_1x02_P2.54mm_Vertical" (layer "F.Cu")
-    (at 78.74 88.646)
+    (at 79.248 100.838)
     (descr "Through hole straight socket strip, 1x02, 2.54mm pitch, single row (from Kicad 4.0.7), script generated")
     (tags "Through hole socket strip THT 1x02 2.54mm single row")
@@
     )
   )
-  (footprint "Connector_PinHeader_2.54mm:PinHeader_1x04_P2.54mm_Vertical" (layer "F.Cu")
+  (footprint "Connector_PinSocket_2.54mm:PinSocket_1x04_P2.54mm_Vertical" (layer "F.Cu")
     (at 145.879 79.655)
-    (descr "Through hole straight pin header, 1x04, 2.54mm pitch, single row")
-    (tags "Through hole pin header THT 1x04 2.54mm single row")
+    (descr "Through hole straight socket strip, 1x04, 2.54mm pitch, single row (from Kicad 4.0.7), script generated")
+    (tags "Through hole socket strip THT 1x04 2.54mm single row")
     (property "Sheetfile" "MaisonEtape1.kicad_sch")
     (property "Sheetname" "")
@@
     (property "ki_keywords" "connector")
     (attr through_hole)
-    (fp_text reference "J_U2" (at 0 -2.33) (layer "F.SilkS")
+    (fp_text reference "J_U2" (at 0 -2.77) (layer "F.SilkS") hide
         (effects (font (size 1 1) (thickness 0.15)))
     )
-    (fp_text value "Conn_01x04_Socket" (at 0 9.95) (layer "F.Fab")
+    (fp_text value "Conn_01x04_Socket" (at 0 10.39) (layer "F.Fab") hide
         (effects (font (size 1 1) (thickness 0.15)))
     )
@@
         (effects (font (size 1 1) (thickness 0.15)))
     )
-    (fp_line (start -1.33 -1.33) (end 0 -1.33)
-      (stroke (width 0.12) (type solid)) (layer "F.SilkS"))
-    (fp_line (start -1.33 0) (end -1.33 -1.33)
-      (stroke (width 0.12) (type solid)) (layer "F.SilkS"))
     (fp_line (start -1.33 1.27) (end -1.33 8.95)
       (stroke (width 0.12) (type solid)) (layer "F.SilkS"))
@@
     (fp_line (start -1.33 8.95) (end 1.33 8.95)
       (stroke (width 0.12) (type solid)) (layer "F.SilkS"))
+    (fp_line (start 0 -1.33) (end 1.33 -1.33)
+      (stroke (width 0.12) (type solid)) (layer "F.SilkS"))
+    (fp_line (start 1.33 -1.33) (end 1.33 0)
+      (stroke (width 0.12) (type solid)) (layer "F.SilkS"))
     (fp_line (start 1.33 1.27) (end 1.33 8.95)
       (stroke (width 0.12) (type solid)) (layer "F.SilkS"))
-    (fp_line (start -1.8 -1.8) (end -1.8 9.4)
+    (fp_line (start -1.8 -1.8) (end 1.75 -1.8)
       (stroke (width 0.05) (type solid)) (layer "F.CrtYd"))
-    (fp_line (start -1.8 9.4) (end 1.8 9.4)
+    (fp_line (start -1.8 9.4) (end -1.8 -1.8)
       (stroke (width 0.05) (type solid)) (layer "F.CrtYd"))
-    (fp_line (start 1.8 -1.8) (end -1.8 -1.8)
+    (fp_line (start 1.75 -1.8) (end 1.75 9.4)
       (stroke (width 0.05) (type solid)) (layer "F.CrtYd"))
-    (fp_line (start 1.8 9.4) (end 1.8 -1.8)
+    (fp_line (start 1.75 9.4) (end -1.8 9.4)
       (stroke (width 0.05) (type solid)) (layer "F.CrtYd"))
-    (fp_line (start -1.27 -0.635) (end -0.635 -1.27)
+    (fp_line (start -1.27 -1.27) (end 0.635 -1.27)
       (stroke (width 0.1) (type solid)) (layer "F.Fab"))
-    (fp_line (start -1.27 8.89) (end -1.27 -0.635)
+    (fp_line (start -1.27 8.89) (end -1.27 -1.27)
       (stroke (width 0.1) (type solid)) (layer "F.Fab"))
-    (fp_line (start -0.635 -1.27) (end 1.27 -1.27)
+    (fp_line (start 0.635 -1.27) (end 1.27 -0.635)
       (stroke (width 0.1) (type solid)) (layer "F.Fab"))
-    (fp_line (start 1.27 -1.27) (end 1.27 8.89)
+    (fp_line (start 1.27 -0.635) (end 1.27 8.89)
       (stroke (width 0.1) (type solid)) (layer "F.Fab"))
     (fp_line (start 1.27 8.89) (end -1.27 8.89)
@@
     (pad "4" thru_hole oval (at 0 7.62) (size 1.7 1.7) (drill 1) (layers "*.Cu" "*.Mask")
       (net 38 "U2_i2c_SDA") (pinfunction "Pin_4") (pintype "passive"))
-    (model "${KICAD6_3DMODEL_DIR}/Connector_PinHeader_2.54mm.3dshapes/PinHeader_1x04_P2.54mm_Vertical.wrl"
+    (model "${KICAD6_3DMODEL_DIR}/Connector_PinSocket_2.54mm.3dshapes/PinSocket_1x04_P2.54mm_Vertical.wrl"
       (offset (xyz 0 0 0))
       (scale (xyz 1 1 1))
@@
   (gr_poly
     (pts
+      (xy 141.986 110.283908)
+      (xy 141.986 111.252)
+      (xy 105.537 111.252)
+      (xy 105.537 110.283908)
+    )
+    (stroke (width 0.1) (type solid)) (fill solid) (layer "Edge.Cuts"))
+  (gr_poly
+    (pts
       (xy 141.224 74.495908)
       (xy 141.224 75.464)
@@
   (gr_poly
     (pts
+      (xy 141.986 128.063908)
+      (xy 141.986 129.032)
+      (xy 105.283 129.032)
+      (xy 105.283 128.063908)
+    )
+    (stroke (width 0.1) (type solid)) (fill solid) (layer "Edge.Cuts"))
+  (gr_poly
+    (pts
       (xy 141.224 92.275908)
       (xy 141.224 93.244)
@@
     (effects (font (size 0.6 0.6) (thickness 0.12) bold) (justify left bottom))
   )
+  (gr_text "SCK\n" (at 148.082 117.348) (layer "F.SilkS")
+    (effects (font (size 1 1) (thickness 0.2) bold) (justify left bottom))
+  )
   (gr_text "SCK\n" (at 133.814 43.46 90) (layer "F.SilkS")
     (effects (font (size 0.6 0.6) (thickness 0.12) bold) (justify left bottom))
@@
     (effects (font (size 0.6 0.6) (thickness 0.12) bold) (justify left bottom))
   )
+  (gr_text "CS1" (at 148.082 114.808) (layer "F.SilkS")
+    (effects (font (size 1 1) (thickness 0.2) bold) (justify left bottom))
+  )
   (gr_text "MOSI" (at 148.082 106.706) (layer "F.SilkS")
     (effects (font (size 1 1) (thickness 0.2) bold) (justify left bottom))
@@
     )
   )
+  (gr_text "MOSI" (at 148.082 122.682) (layer "F.SilkS")
+    (effects (font (size 1 1) (thickness 0.2) bold) (justify left bottom))
+  )
   (gr_text "TX" (at 149.054 43.46 90) (layer "F.SilkS")
     (effects (font (size 0.6 0.6) (thickness 0.12) bold) (justify left bottom))
@@
     (effects (font (size 0.6 0.6) (thickness 0.12) bold) (justify left bottom))
   )
+  (gr_text "MISO" (at 148.082 120.142) (layer "F.SilkS")
+    (effects (font (size 1 1) (thickness 0.2) bold) (justify left bottom))
+  )
   (gr_text "RX" (at 151.594 43.46 90) (layer "F.SilkS")

Commit message: update friday pcb
Parts:
- added BZ1: Buzzer, Buzzer_Beeper:Buzzer_12x9.5RM7.6, F.Cu at (108.6, 131.4)
- added J10: Conn_01x13_Pin, Connector_PinHeader_2.54mm:PinHeader_1x13_P2.54mm_Vertical, F.Cu at (174.6, 125.1)
- added SW6: SW_SPDT, JPLibrary:BSI-10, F.Cu at (68.2, 47.5)
- added SW7: SW_SPDT, JPLibrary:BSI-10, F.Cu at (124.5, 137.2)
- added U6: 4021, Package_DIP:DIP-16_W7.62mm_LongPads, F.Cu at (152.4, 130.2)
- added U7: 4021, Package_DIP:DIP-16_W7.62mm_LongPads, F.Cu at (175.3, 130.2)
- J1, J2, J3, Jmaster1: footprint Connector_IDC:IDC-Header_2x03_P2.54mm_Vertical -> JPLibrary:SPI_prog
- J4: renamed from J13; footprint Connector_IDC:IDC-Header_2x03_P2.54mm_Vertical -> JPLibrary:SPI_prog
- J5: renamed from J4; footprint Connector_IDC:IDC-Header_2x03_P2.54mm_Vertical -> JPLibrary:SPI_prog
- J_SPI_5: footprint Connector:NS-Tech_Grove_1x04_P2mm_Vertical -> Connector_PinHeader_2.54mm:PinHeader_1x04_P2.54mm_Vertical
- SW5: footprint Button_Switch_THT:SW_E-Switch_EG1271_SPDT -> JPLibrary:BSI-10
- moved J_SPI_5 114.6 mm to (180.3, 129.8)
- moved J4 86.6 mm to (106.0, 113.7)
- moved Q2 69.0 mm to (128.3, 118.1)
- moved J5 67.8 mm to (100.3, 128.3)
- moved J12 51.1 mm to (129.5, 109.9), turned to 90 degrees
- moved U5 45.8 mm to (126.1, 129.3)
- moved U4 9.08 mm to (117.8, 113.9)
- moved J11 8.55 mm to (129.2, 93.4)
- moved J_SPI_3 8.55 mm to (139.3, 93.4)
- moved U3 8.55 mm to (118.3, 97.0)
- moved Q1 7.51 mm to (127.6, 101.6)
- moved J_SPI_4 7.41 mm to (139.7, 110.5)
- moved R17 7.21 mm to (125.5, 84.6)
- moved Door1 7.21 mm to (130.2, 77.3)
- moved J_U2 7.21 mm to (139.1, 77.3)
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- renumbered J5 to J13
Other:
- board size 100 x 100 mm -> 96.8 x 99.4 mm
