File: kicad/Sheet_clavier.kicad_sch (KiCad schematic)
At the start: 15 parts, among them U6 4021, U7 4021

Commit message: update sur tout le schema
Parts:
- added J10: Conn_01x13_Pin, symbol Connector:Conn_01x13_Pin
- CLAVIER2: now left out of the parts list
Connections:
- net +5V: now also J10.1 (Pin_1)
- net QA1: now also J10.6 (Pin_6); no longer CLAVIER2.0
- net QA2: now also J10.7 (Pin_7); no longer CLAVIER2.8
- net QB1: now also J10.5 (Pin_5); no longer CLAVIER2.1
- net QB2: now also J10.11 (Pin_11); no longer CLAVIER2.9
- net QC1: now also J10.9 (Pin_9); no longer CLAVIER2.2
- net QC2: now also J10.2 (Pin_2); no longer CLAVIER2.*
- net QD1: now also J10.13 (Pin_13); no longer CLAVIER2.3
- net QD2: now also J10.10 (Pin_10); no longer CLAVIER2.#
- net QE1: now also J10.4 (Pin_4); no longer CLAVIER2.4
- net QF1: now also J10.8 (Pin_8); no longer CLAVIER2.5
- net QG1: now also J10.12 (Pin_12); no longer CLAVIER2.6
- net QH1: now also J10.3 (Pin_3); no longer CLAVIER2.7
Other:
- note added: "#"
- note added: "*"
- note added: "0"
- note added: "1"
- note added: "2"
- note added: "3"
- note added: "4"
- note added: "5"
- note added: "6"
- note added: "7"
- note added: "8"
- note added: "9"
- moved on the sheet: CLAVIER2

Commit message: updates clavier
Connections:
- net GND: now also U6.14 (P5), U6.15 (P6); no longer U7.1 (P7), U7.13 (P4)
- net QA1: now also J10.13 (Pin_13), R14.2; no longer J10.6 (Pin_6), R7.2
- net QB1: now also J10.12 (Pin_12), R13.2; no longer J10.5 (Pin_5), R6.2
- net QB2: now also J10.6 (Pin_6), R7.2; no longer J10.11 (Pin_11), R12.2
- net QC1: now also J10.11 (Pin_11), R12.2; no longer J10.9 (Pin_9), R10.2
- net QC2: now also J10.5 (Pin_5), R6.2; no longer J10.2 (Pin_2), R3.2
- net QD1: now also J10.10 (Pin_10), R11.2; no longer J10.13 (Pin_13), R14.2
- net QD2: now also J10.4 (Pin_4), R5.2; no longer J10.10 (Pin_10), R11.2
- net QE1: now also J10.8 (Pin_8), R9.2; no longer J10.4 (Pin_4), R5.2
- net QH1: now also J10.9 (Pin_9), R10.2; no longer J10.3 (Pin_3), R4.2
- removed net QF1: J10.8 (Pin_8), R9.2, U6.14 (P5)
- removed net QG1: J10.12 (Pin_12), R13.2, U6.15 (P6)
- new net QE2: J10.2 (Pin_2), R3.2, U7.13 (P4)
- new net QH2: J10.3 (Pin_3), R4.2, U7.1 (P7)
Other:
- note added: "0x1"
- note added: "0x10"
- note added: "0x100"
- note added: "0x1000"
- note added: "0x20"
- note added: "0x2000"
- note added: "0x40"
- note added: "0x4000"
- note added: "0x8"
- note added: "0x80"
- note added: "0x800"
- note added: "0x8000"
- note added: "[1]"
- note added: "[2]"

Commit message: update friday pcb
Parts:
- J10: footprint (none) -> Connector_PinHeader_2.54mm:PinHeader_1x13_P2.54mm_Vertical
- U6, U7: footprint (none) -> Package_DIP:DIP-16_W7.62mm_LongPads
Changed lines of the file:
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@@
       (effects (font (size 1.27 1.27)) (justify left))
     )
-    (property "Footprint" "" (at 203.2 118.11 0)
+    (property "Footprint" "Package_DIP:DIP-16_W7.62mm_LongPads" (at 203.2 118.11 0)
       (effects (font (size 1.27 1.27)) hide)
     )
@@
       (effects (font (size 1.27 1.27)) (justify left))
     )
-    (property "Footprint" "" (at 204.47 63.5 0)
+    (property "Footprint" "Package_DIP:DIP-16_W7.62mm_LongPads" (at 204.47 63.5 0)
       (effects (font (size 1.27 1.27)) hide)
     )
@@
       (effects (font (size 1.27 1.27)))
     )
-    (property "Footprint" "" (at 102.87 88.9 0)
-      (effects (font (size 1.27 1.27)) hide)
-    )
+    (property "Footprint" "Connector_PinHeader_2.54mm:PinHeader_1x13_P2.54mm_Vertical" (at 102.87 88.9 0)
+      (effects (font (size 1.27 1.27)) hide)
+    )

Commit message: kicad update, finalizing
Parts:
- R10, R11, R12, R13, R14, R3, R4, R5, R6, R7, R8, R9: footprint (none) -> Resistor_SMD:R_0805_2012Metric_Pad1.20x1.40mm_HandSolder
Connections:
- net +5V: no longer J10.1 (Pin_1), U6.16 (Vdd), U7.16 (Vdd)
- net GND renamed U5_GND
- new net U5_VCC: J10.1 (Pin_1), U6.16 (Vdd), U7.16 (Vdd)
