File: kicad/untitled.kicad_sch (KiCad schematic)
At the start: 10 parts, among them J3 AVR-ISP-6, J4 AVR-ISP-6, J5 AVR-ISP-6, M1 Motor_DC, Q1 NMOS, U3 ATmega328P-P, U4 ATmega328P-P, U5 ATmega328P-P

Commit message: update sur tout le schema
Parts:
- removed J5: AVR-ISP-6, Connector_IDC:IDC-Header_2x03_P2.54mm_Vertical, symbol Connector:AVR-ISP-6
- added J11, J12: Conn_01x02_Socket, symbol Connector:Conn_01x02_Socket
- added J13: AVR-ISP-6, Connector_IDC:IDC-Header_2x03_P2.54mm_Vertical, symbol Connector:AVR-ISP-6
- added J6, J7, J8, J9: Conn_01x01_Pin, symbol Connector:Conn_01x01_Pin
- added LA1: Lamp, symbol Device:Lamp
- added Q2: NMOS, symbol Simulation_SPICE:NMOS
- added R18: 1K, symbol Device:R
- added R19: 200R, symbol Device:R
- added SW4 (x3): SW_SPDT, symbol Switch:SW_SPDT
- M1: now left out of the parts list
Connections:
- net +5V: now also U3.20 (AVCC), U4.20 (AVCC), U5.20 (AVCC), J11.1 (Pin_1), J12.1 (Pin_1), J13.2 (VCC); no longer M1.1 (+)
- net CS: now also SW4.3 (C), SW4.3 (C), SW4.3 (C); no longer U3.16 (PB2), U4.16 (PB2), U5.16 (PB2)
- net Clavier_latchPin: now also U5.2 (PD0); no longer U5.14 (PB0)
- net GND: now also J13.6 (GND), Q2.3 (S), R19.1
- net GPIO_Moteur: now also U4.28 (PC5)
- net SPI_MISO: now also J3.1 (MISO), J4.1 (MISO), J13.1 (MISO)
- net SPI_MOSI: now also J3.4 (MOSI), J4.4 (MOSI), J13.4 (MOSI)
- net at U3.1 (~{RESET}/PC6): now also J3.5 (~{RST})
- net SPI_SCK: now reaches U3.19 (PB5)
- net SPI_SCK: now also J3.3 (SCK), J4.3 (SCK), U4.19 (PB5), U5.19 (PB5), J13.3 (SCK)
- net GPIO_Lumiere: now reaches U3.28 (PC5)
- net GPIO_Lumiere: now also R18.1
- net at U4.1 (~{RESET}/PC6): now also J13.5 (~{RST})
- net at Q1.1 (D): now also J11.2 (Pin_2); no longer M1.2 (-)
- net at U5.1 (~{RESET}/PC6): now also J4.5 (~{RST})
- new net: J7.1 (Pin_1), LA1.1 (-)
- new net: J6.1 (Pin_1), LA1.2 (+)
- new net: SW4.2 (B), U4.16 (PB2)
- new net: SW4.2 (B), U3.16 (PB2)
- new net: J12.2 (Pin_2), Q2.1 (D)
- new net: Q2.2 (G), R18.2, R19.2
- new net: J9.1 (Pin_1), M1.2 (-)
- new net: SW4.2 (B), U5.16 (PB2)
- new net: J8.1 (Pin_1), M1.1 (+)
Other:
- note added: "LUMIERE"
- moved on the sheet: Q1, R1, R2, U3, U4, U5

Commit message: updates clavier
Parts:
- added BZ1: Buzzer, symbol Device:Buzzer
Connections:
- net Clavier_clockPin: now also U5.24 (PC1); no longer U5.4 (PD2)
- net Clavier_dataPin: now also U5.25 (PC2); no longer U5.11 (PD5)
- net Clavier_latchPin: now also U5.23 (PC0); no longer U5.2 (PD0)
- net GND: now also BZ1.2 (+)
- net at U5.26 (PC3): now also BZ1.1 (-)
Changed lines of the file:
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@@
+    (stroke (width 0) (type default))
+  )
+  (wire (pts (xy 232.41 127) (xy 232.41 107.95))
     (stroke (width 0) (type default))
   )
@@
     (stroke (width 0) (type default))
   )
+  (wire (pts (xy 231.14 129.54) (xy 231.14 110.49))
+    (stroke (width 0) (type default))
+  )
   (wire (pts (xy 167.64 100.33) (xy 167.64 123.19))
     (stroke (width 0) (type default))
   )
+  (wire (pts (xy 228.6 115.57) (xy 241.3 115.57))
+    (stroke (width 0) (type default))
+  )
   (wire (pts (xy 43.18 73.66) (xy 40.64 73.66))
     (stroke (width 0) (type default))
@@
     (stroke (width 0) (type default))
   )
+  (wire (pts (xy 229.87 132.08) (xy 229.87 113.03))
+    (stroke (width 0) (type default))
+  )
   (wire (pts (xy 63.5 53.34) (xy 67.31 53.34))
     (stroke (width 0) (type default))
@@
     (stroke (width 0) (type default))
   )
+  (wire (pts (xy 236.22 127) (xy 232.41 127))
+    (stroke (width 0) (type default))
+  )
   (wire (pts (xy 228.6 90.17) (xy 236.22 90.17))
     (stroke (width 0) (type default))
@@
     (stroke (width 0) (type default))
   )
+  (wire (pts (xy 236.22 132.08) (xy 229.87 132.08))
+    (stroke (width 0) (type default))
+  )
   (wire (pts (xy 158.75 92.71) (xy 167.64 92.71))
     (stroke (width 0) (type default))
@@
     (stroke (width 0) (type default))
   )
+  (wire (pts (xy 229.87 113.03) (xy 228.6 113.03))
+    (stroke (width 0) (type default))
+  )
   (wire (pts (xy 160.02 63.5) (xy 160.02 66.04))
     (stroke (width 0) (type default))
@@
     (stroke (width 0) (type default))
   )
+  (wire (pts (xy 232.41 107.95) (xy 228.6 107.95))
+    (stroke (width 0) (type default))
+  )
   (wire (pts (xy 73.66 91.44) (xy 81.28 91.44))
     (stroke (width 0) (type default))
   )
+  (wire (pts (xy 236.22 129.54) (xy 231.14 129.54))
+    (stroke (width 0) (type default))
+  )
   (wire (pts (xy 160.02 58.42) (xy 160.02 63.5))
     (stroke (width 0) (type default))
@@
   )
   (wire (pts (xy 245.11 100.33) (xy 245.11 92.71))
+    (stroke (width 0) (type default))
+  )
+  (wire (pts (xy 231.14 110.49) (xy 228.6 110.49))
     (stroke (width 0) (type default))
   )
@@
     )
   )
-  (global_label "Clavier_clockPin" (shape input) (at 228.6 133.35 0) (fields_autoplaced)
+  (global_label "Clavier_clockPin" (shape input) (at 236.22 129.54 0) (fields_autoplaced)
     (effects (font (size 1.27 1.27)) (justify left))
-    (property "Intersheetrefs" "${INTERSHEET_REFS}" (at 247.0481 133.35 0)
+    (property "Intersheetrefs" "${INTERSHEET_REFS}" (at 254.6681 129.54 0)
       (effects (font (size 1.27 1.27)) (justify left) hide)
     )
@@
     )
   )
-  (global_label "Clavier_latchPin" (shape input) (at 228.6 128.27 0) (fields_autoplaced)
+  (global_label "Clavier_latchPin" (shape input) (at 236.22 127 0) (fields_autoplaced)
     (effects (font (size 1.27 1.27)) (justify left))
-    (property "Intersheetrefs" "${INTERSHEET_REFS}" (at 246.8061 128.27 0)
+    (property "Intersheetrefs" "${INTERSHEET_REFS}" (at 254.4261 127 0)
       (effects (font (size 1.27 1.27)) (justify left) hide)
     )
@@
     )
   )
-  (global_label "Clavier_dataPin" (shape input) (at 228.6 140.97 0) (fields_autoplaced)
+  (global_label "Clavier_dataPin" (shape input) (at 236.22 132.08 0) (fields_autoplaced)
     (effects (font (size 1.27 1.27)) (justify left))
-    (property "Intersheetrefs" "${INTERSHEET_REFS}" (at 246.2013 140.97 0)
+    (property "Intersheetrefs" "${INTERSHEET_REFS}" (at 253.8213 132.08 0)
       (effects (font (size 1.27 1.27)) (justify left) hide)
     )
@@
     )
   )
+  (symbol (lib_id "power:GND") (at 241.3 120.65 270) (unit 1)
+    (in_bom yes) (on_board yes) (dnp no) (fields_autoplaced)
+    (property "Reference" "#PWR049" (at 234.95 120.65 0)
+      (effects (font (size 1.27 1.27)) hide)
+    )
+    (property "Value" "GND" (at 237.49 120.65 90)
+      (effects (font (size 1.27 1.27)) (justify right))
+    )
+    (property "Footprint" "" (at 241.3 120.65 0)
+      (effects (font (size 1.27 1.27)) hide)
+    )
+    (property "Datasheet" "" (at 241.3 120.65 0)
+      (effects (font (size 1.27 1.27)) hide)
+    )
+    (pin "1")
+    (instances
+      (project "MaisonEtape1"
+        (path "/ed06f8de-d1bb-4b1a-bfe3-5df11d3a9162"
+          (reference "#PWR049") (unit 1)
+        )
+        (path "/ed06f8de-d1bb-4b1a-bfe3-5df11d3a9162/0600536b-f413-4b06-98e9-b5748b5de992"
+          (reference "#PWR055") (unit 1)
+        )
+      )
+    )
+  )
   (symbol (lib_id "MCU_Microchip_ATmega:ATmega328P-P") (at 127 115.57 0) (unit 1)
     (in_bom yes) (on_board yes) (dnp no)
@@
         )
       )
+    )
+  )
+  (symbol (lib_id "Device:Buzzer") (at 243.84 118.11 0) (unit 1)
+    (in_bom yes) (on_board yes) (dnp no)
+    (property "Reference" "BZ1" (at 247.65 116.84 0)
+      (effects (font (size 1.27 1.27)) (justify left))
+    )
+    (property "Value" "Buzzer" (at 246.38 120.65 0)
+      (effects (font (size 1.27 1.27)) (justify left))
+    )
+    (property "Footprint" "" (at 243.205 115.57 90)
+      (effects (font (size 1.27 1.27)) hide)
+    )
+    (property "Datasheet" "~" (at 243.205 115.57 90)
+      (effects (font (size 1.27 1.27)) hide)
+    )
+    (pin "1")
+    (pin "2")
+    (instances
+      (project "MaisonEtape1"
+        (path "/ed06f8de-d1bb-4b1a-bfe3-5df11d3a9162/0600536b-f413-4b06-98e9-b5748b5de992"
+          (reference "BZ1") (unit 1)
+        )
+      )

Commit message: lfg
Connections:
- removed net CS: SW4.3 (C), SW4.3 (C), SW4.3 (C)
- new net CS1: SW4.3 (C)
- new net CS2: SW4.3 (C)
- new net CS3: SW4.3 (C)
Changed lines of the file:
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@@
     )
   )
-  (global_label "CS" (shape input) (at 76.2 88.9 0) (fields_autoplaced)
+  (global_label "CS1" (shape input) (at 76.2 88.9 0) (fields_autoplaced)
     (effects (font (size 1.27 1.27)) (justify left))
-    (property "Intersheetrefs" "${INTERSHEET_REFS}" (at 81.5853 88.9 0)
+    (property "Intersheetrefs" "${INTERSHEET_REFS}" (at 82.8742 88.9 0)
       (effects (font (size 1.27 1.27)) (justify left) hide)
     )
@@
     )
   )
-  (global_label "CS" (shape input) (at 248.92 90.17 0) (fields_autoplaced)
+  (global_label "CS3" (shape input) (at 248.92 90.17 0) (fields_autoplaced)
     (effects (font (size 1.27 1.27)) (justify left))
-    (property "Intersheetrefs" "${INTERSHEET_REFS}" (at 254.3053 90.17 0)
+    (property "Intersheetrefs" "${INTERSHEET_REFS}" (at 255.5942 90.17 0)
       (effects (font (size 1.27 1.27)) (justify left) hide)
     )
@@
     )
   )
-  (global_label "CS" (shape input) (at 162.56 90.17 0) (fields_autoplaced)
+  (global_label "CS2" (shape input) (at 162.56 90.17 0) (fields_autoplaced)
     (effects (font (size 1.27 1.27)) (justify left))
-    (property "Intersheetrefs" "${INTERSHEET_REFS}" (at 167.9453 90.17 0)
+    (property "Intersheetrefs" "${INTERSHEET_REFS}" (at 169.2342 90.17 0)
       (effects (font (size 1.27 1.27)) (justify left) hide)
     )

Commit message: 13-10
Parts:
- removed U3, U4, U5: ATmega328P-P, Package_DIP:DIP-28_W7.62mm, symbol MCU_Microchip_ATmega:ATmega328P-P
- added J_SPI_3, J_SPI_4, J_SPI_5: SPI_SOCKET, Connector:NS-Tech_Grove_1x04_P2mm_Vertical, symbol Connector:Conn_01x04_Socket
- added U3, U4, U5: ATmega8A-A, Package_QFP:TQFP-32_7x7mm_P0.8mm, symbol MCU_Microchip_ATmega:ATmega8A-A
Connections:
- net +5V: now also U3.18 (AVCC), U3.4 (VCC), U3.6 (VCC), U4.18 (AVCC), U4.4 (VCC), U4.6 (VCC), U5.18 (AVCC), U5.4 (VCC), U5.6 (VCC)
- net Clavier_clockPin: now also U5.24 (PC1)
- net Clavier_dataPin: now also U5.25 (PC2)
- net Clavier_latchPin: now also U5.23 (PC0)
- net GND: now also U3.3 (GND), U3.5 (GND), U4.3 (GND), U4.5 (GND), U5.21 (AGND)
- net GPIO_Lumiere: now also U3.28 (PC5)
- net GPIO_Moteur: now also U4.28 (PC5)
- net at SW4.2 (B): now also U4.14 (PB2)
- net U3_RESET: now reaches J3.5 (~{RST})
- net U3_RESET: now also U3.29 (PC6/~{RESET})
- net at SW4.2 (B): now also U3.14 (PB2)
- net U4_RESET: now reaches J13.5 (~{RST})
- net U4_RESET: now also U4.29 (PC6/~{RESET})
- net U5_RESET: now reaches J4.5 (~{RST})
- net U5_RESET: now also U5.29 (PC6/~{RESET})
- net at BZ1.1 (-): now also U5.26 (PC3)
- net at SW4.2 (B): now also U5.14 (PB2)
- net CS1 renamed U3_CS1
- net U3_CS1: now also J_SPI_3.1 (Pin_1)
- net CS2 renamed U4_CS2
- net U4_CS2: now also J_SPI_4.1 (Pin_1)
- net CS3 renamed U5_CS3
- net U5_CS3: now also J_SPI_5.1 (Pin_1)
- removed net SPI_MISO: J13.1 (MISO), J3.1 (MISO), J4.1 (MISO)
- removed net SPI_MOSI: J13.4 (MOSI), J3.4 (MOSI), J4.4 (MOSI)
- removed net SPI_SCK: J13.3 (SCK), J3.3 (SCK), J4.3 (SCK)
- new net: U5.3 (GND), U5.5 (GND)
- new net U3_SPI_MISO: J3.1 (MISO), J_SPI_3.3 (Pin_3), U3.16 (PB4)
- new net U3_SPI_MOSI: J3.4 (MOSI), J_SPI_3.4 (Pin_4), U3.15 (PB3)
- new net U3_SPI_SCK: J3.3 (SCK), J_SPI_3.2 (Pin_2), U3.17 (PB5)
- new net U4_SPI_MISO: J13.1 (MISO), J_SPI_4.3 (Pin_3), U4.16 (PB4)
- new net U4_SPI_MOSI: J13.4 (MOSI), J_SPI_4.4 (Pin_4), U4.15 (PB3)
- new net U4_SPI_SCK: J13.3 (SCK), J_SPI_4.2 (Pin_2), U4.17 (PB5)
- new net U5_SPI_MISO: J4.1 (MISO), J_SPI_5.3 (Pin_3), U5.16 (PB4)
- new net U5_SPI_MOSI: J4.4 (MOSI), J_SPI_5.4 (Pin_4), U5.15 (PB3)
- new net U5_SPI_SCK: J4.3 (SCK), J_SPI_5.2 (Pin_2), U5.17 (PB5)
Other:
- moved on the sheet: J13, SW4

Commit message: update kicad
Parts:
- J11, J12: footprint (none) -> Connector_PinSocket_2.54mm:PinSocket_1x02_P2.54mm_Vertical
- J_SPI_3, J_SPI_4: footprint Connector:NS-Tech_Grove_1x04_P2mm_Vertical -> Connector_PinHeader_2.54mm:PinHeader_1x04_P2.54mm_Vertical
- Q1, Q2: footprint (none) -> Package_TO_SOT_THT:TO-220-3_Vertical
- R1, R18, R19, R2: footprint (none) -> Resistor_SMD:R_0805_2012Metric_Pad1.20x1.40mm_HandSolder
- SW4: footprint (none) -> Button_Switch_THT:SW_E-Switch_EG1271_SPDT
Connections:
- net +5V: no longer J11.1 (Pin_1), J12.1 (Pin_1), U3.18 (AVCC), U3.4 (VCC), U3.6 (VCC), U4.18 (AVCC), U4.4 (VCC), U4.6 (VCC), U5.18 (AVCC), U5.4 (VCC), U5.6 (VCC)
- net GND: no longer Q1.3 (S), Q2.3 (S), R1.1, R19.1, U3.3 (GND), U3.5 (GND), U4.3 (GND), U4.5 (GND), U5.21 (AGND)
- new net U3_GND: Q2.3 (S), R19.1, U3.3 (GND), U3.5 (GND)
- new net U3_VCC: J12.1 (Pin_1), U3.18 (AVCC), U3.4 (VCC), U3.6 (VCC)
- new net U4_GND: Q1.3 (S), R1.1, U4.3 (GND), U4.5 (GND)
- new net U4_VCC: J11.1 (Pin_1), U4.18 (AVCC), U4.4 (VCC), U4.6 (VCC)
- new net U5_GND: U5.21 (AGND)
- new net U5_VCC: U5.18 (AVCC), U5.4 (VCC), U5.6 (VCC)

Commit message: update friday pcb
Parts:
- BZ1: footprint (none) -> Buzzer_Beeper:Buzzer_12x9.5RM7.6
- J3: footprint Connector_IDC:IDC-Header_2x03_P2.54mm_Vertical -> JPLibrary:SPI_prog
- J4: renamed from J13; footprint Connector_IDC:IDC-Header_2x03_P2.54mm_Vertical -> JPLibrary:SPI_prog
- J5: renamed from J4; footprint Connector_IDC:IDC-Header_2x03_P2.54mm_Vertical -> JPLibrary:SPI_prog
- SW4: footprint (none) -> JPLibrary:BSI-10
- SW4: footprint Button_Switch_THT:SW_E-Switch_EG1271_SPDT -> JPLibrary:BSI-10
Changed lines of the file:
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@@
     (stroke (width 0) (type default))
   )
-  (wire (pts (xy 210.82 74.93) (xy 210.82 73.66))
+  (wire (pts (xy 210.82 74.93) (xy 210.82 66.04))
     (stroke (width 0) (type default))
   )
@@
     )
   )
-  (global_label "U5_VCC" (shape input) (at 210.82 73.66 0) (fields_autoplaced)
-    (effects (font (size 1.27 1.27)) (justify left))
-    (property "Intersheetrefs" "${INTERSHEET_REFS}" (at 220.9414 73.66 0)
+  (global_label "U5_VCC" (shape input) (at 210.82 66.04 0) (fields_autoplaced)
+    (effects (font (size 1.27 1.27)) (justify left))
+    (property "Intersheetrefs" "${INTERSHEET_REFS}" (at 220.9414 66.04 0)
       (effects (font (size 1.27 1.27)) (justify left) hide)
     )
@@
       (effects (font (size 1.27 1.27)))
     )
-    (property "Footprint" "" (at 156.845 90.805 0)
+    (property "Footprint" "JPLibrary:BSI-10" (at 156.845 90.805 0)
       (effects (font (size 1.27 1.27)) hide)
     )
@@
   (symbol (lib_name "AVR-ISP-6_1") (lib_id "Connector:AVR-ISP-6") (at 264.16 97.79 0) (mirror y) (unit 1)
     (in_bom yes) (on_board yes) (dnp no)
-    (property "Reference" "J4" (at 273.05 95.25 0)
+    (property "Reference" "J5" (at 273.05 95.25 0)
       (effects (font (size 1.27 1.27)) (justify right))
     )
@@
       (effects (font (size 1.27 1.27)) (justify right))
     )
-    (property "Footprint" "Connector_IDC:IDC-Header_2x03_P2.54mm_Vertical" (at 270.51 96.52 90)
+    (property "Footprint" "JPLibrary:SPI_prog" (at 270.51 96.52 90)
       (effects (font (size 1.27 1.27)) hide)
     )
@@
       (project "MaisonEtape1"
         (path "/ed06f8de-d1bb-4b1a-bfe3-5df11d3a9162/0600536b-f413-4b06-98e9-b5748b5de992"
-          (reference "J4") (unit 1)
+          (reference "J5") (unit 1)
         )
         (path "/ed06f8de-d1bb-4b1a-bfe3-5df11d3a9162"
@@
       (effects (font (size 1.27 1.27)) (justify left))
     )
-    (property "Footprint" "" (at 243.205 115.57 90)
+    (property "Footprint" "Buzzer_Beeper:Buzzer_12x9.5RM7.6" (at 243.205 115.57 90)
       (effects (font (size 1.27 1.27)) hide)
     )
@@
       (effects (font (size 1.27 1.27)))
     )
-    (property "Footprint" "" (at 241.3 87.63 0)
+    (property "Footprint" "JPLibrary:BSI-10" (at 241.3 87.63 0)
       (effects (font (size 1.27 1.27)) hide)
     )
@@
       (effects (font (size 1.27 1.27)) (justify right))
     )
-    (property "Footprint" "Connector_IDC:IDC-Header_2x03_P2.54mm_Vertical" (at 97.79 95.25 90)
+    (property "Footprint" "JPLibrary:SPI_prog" (at 97.79 95.25 90)
       (effects (font (size 1.27 1.27)) hide)
     )
@@
       (effects (font (size 1.27 1.27)))
     )
-    (property "Footprint" "Button_Switch_THT:SW_E-Switch_EG1271_SPDT" (at 68.58 86.36 0)
+    (property "Footprint" "JPLibrary:BSI-10" (at 68.58 86.36 0)
       (effects (font (size 1.27 1.27)) hide)
     )
@@
   (symbol (lib_name "AVR-ISP-6_1") (lib_id "Connector:AVR-ISP-6") (at 181.61 100.33 0) (mirror y) (unit 1)
     (in_bom yes) (on_board yes) (dnp no)
-    (property "Reference" "J13" (at 190.5 97.79 0)
+    (property "Reference" "J4" (at 190.5 97.79 0)
       (effects (font (size 1.27 1.27)) (justify right))
     )
@@
       (effects (font (size 1.27 1.27)) (justify right))
     )
-    (property "Footprint" "Connector_IDC:IDC-Header_2x03_P2.54mm_Vertical" (at 187.96 99.06 90)
+    (property "Footprint" "JPLibrary:SPI_prog" (at 187.96 99.06 90)
       (effects (font (size 1.27 1.27)) hide)
     )
@@
       (project "MaisonEtape1"
         (path "/ed06f8de-d1bb-4b1a-bfe3-5df11d3a9162/0600536b-f413-4b06-98e9-b5748b5de992"
-          (reference "J13") (unit 1)
+          (reference "J4") (unit 1)
         )
         (path "/ed06f8de-d1bb-4b1a-bfe3-5df11d3a9162"

Commit message: kicad update, finalizing
Parts:
- removed J6, J7, J8, J9: Conn_01x01_Pin, symbol Connector:Conn_01x01_Pin
- removed LA1: Lamp, symbol Device:Lamp
- removed M1: Motor_DC, symbol Motor:Motor_DC
- added C1, C2, C3, C4, C5, C6: 16pF, Capacitor_SMD:C_0805_2012Metric_Pad1.18x1.45mm_HandSolder, symbol Device:C
- added R29 (x2): 220, Resistor_SMD:R_0805_2012Metric_Pad1.20x1.40mm_HandSolder, symbol Device:R
- added U3_PW1, U4_PW1, U5_PW1: Conn_01x03_MountingPin, Connector_PinHeader_2.54mm:PinHeader_1x02_P2.54mm_Vertical, symbol Connector_Generic:Conn_01x02
- added U3_XT_L1, U3_XT_R1, U4_XT_L1, U4_XT_R1: Conn_01x08, JP_Library:XT_8, symbol Connector_Generic:Conn_01x08
- added U5_XT1: Conn_01x14, JP_Library:XT_14, symbol Connector_Generic:Conn_01x14
- added Window_1 (x2): LED, LED_SMD:LED_0805_2012Metric, symbol Device:LED
- added Y_U3, Y_U4, Y_U5: Crystal, JP_Library:Crystal 49SS-SMD, symbol Device:Crystal
- J_SPI_5: footprint Connector:NS-Tech_Grove_1x04_P2mm_Vertical -> Connector_PinHeader_2.54mm:PinHeader_1x04_P2.54mm_Vertical
- SW4: footprint JPLibrary:BSI-10 -> JP_Library:BSI-10; symbol Switch:SW_SPDT -> JP_Library:BSI-10
Connections:
- net U3_CS1: now also SW4.2 (cs); no longer SW4.3 (C)
- net U3_GND: now also J3.6 (GND), U3.21 (AGND), C3.2, C4.2, U3_PW1.2 (Pin_2), Window_1.1 (K)
- net U3_VCC: now also J3.2 (VCC), U3_PW1.1 (Pin_1)
- net U4_CS2: now also SW4.2 (cs); no longer SW4.3 (C)
- net U4_GND: now also J4.6 (GND), U4.21 (AGND), C1.2, C2.2, U4_PW1.2 (Pin_2), Window_1.1 (K)
- net U4_VCC: now also J4.2 (VCC), U4_PW1.1 (Pin_1)
- net U5_CS3: now also SW4.2 (cs); no longer SW4.3 (C)
- net U5_GND: now also BZ1.2 (+), J5.6 (GND), U5.3 (GND), U5.5 (GND), C5.2, C6.2, U5_PW1.2 (Pin_2)
- net U5_VCC: now also J5.2 (VCC), U5_PW1.1 (Pin_1)
- net at SW4.1: now also U4.14 (PB2)
- net U5_PD3: now reaches U5.1 (PD3)
- net U5_PD3: now also U5_XT1.10 (Pin_10)
- net U5_PD6: now reaches U5.10 (PD6)
- net U5_PD6: now also U5_XT1.13 (Pin_13)
- net U5_PD7: now reaches U5.11 (PD7)
- net U5_PD7: now also U5_XT1.14 (Pin_14)
- net U5_PB0: now reaches U5.12 (PB0)
- net U5_PB0: now also U5_XT1.3 (Pin_3)
- net U5_PB1: now reaches U5.13 (PB1)
- net U5_PB1: now also U5_XT1.4 (Pin_4)
- net at U5.14 (PB2): now also SW4.1; no longer SW4.2 (B)
- net U5_ADC6: now reaches U5.19 (ADC6)
- net U5_ADC6: now also U5_XT1.1 (Pin_1)
- net U5_PD4: now reaches U5.2 (PD4)
- net U5_PD4: now also U5_XT1.11 (Pin_11)
- net U5_ADC7: now reaches U5.22 (ADC7)
- net U5_ADC7: now also U5_XT1.2 (Pin_2)
- net U5_PC4: now reaches U5.27 (PC4)
- net U5_PC4: now also U5_XT1.5 (Pin_5)
- net U5_PC5: now reaches U5.28 (PC5)
- net U5_PC5: now also U5_XT1.6 (Pin_6)
- net U5_PD0: now reaches U5.30 (PD0)
- net U5_PD0: now also U5_XT1.7 (Pin_7)
- net U5_PD1: now reaches U5.31 (PD1)
- net U5_PD1: now also U5_XT1.8 (Pin_8)
- net U5_PD2: now reaches U5.32 (PD2)
- net U5_PD2: now also U5_XT1.9 (Pin_9)
- net U5_PB6: now reaches U5.7 (PB6/XTAL1)
- net U5_PB6: now also C5.1, Y_U5.2
- net U5_PB7: now reaches U5.8 (PB7/XTAL2)
- net U5_PB7: now also C6.1, Y_U5.1
- net U5_PD5: now reaches U5.9 (PD5)
- net U5_PD5: now also U5_XT1.12 (Pin_12)
- net U3_PD3: now reaches U3.1 (PD3)
- net U3_PD3: now also U3_XT_R1.4 (Pin_4)
- net U3_PD6: now reaches U3.10 (PD6)
- net U3_PD6: now also U3_XT_R1.7 (Pin_7)
- net U3_PD7: now reaches U3.11 (PD7)
- net U3_PD7: now also U3_XT_R1.8 (Pin_8)
- net U3_PB0: now reaches U3.12 (PB0)
- net U3_PB0: now also R29.2
- net U3_PB1: now reaches U3.13 (PB1)
- net U3_PB1: now also U3_XT_L1.3 (Pin_3)
- net at U3.14 (PB2): now also SW4.1; no longer SW4.2 (B)
- net U3_ADC6: now reaches U3.19 (ADC6)
- net U3_ADC6: now also U3_XT_L1.1 (Pin_1)
- net U3_PD4: now reaches U3.2 (PD4)
- net U3_PD4: now also U3_XT_R1.5 (Pin_5)
- net U3_ADC7: now reaches U3.22 (ADC7)
- net U3_ADC7: now also U3_XT_L1.2 (Pin_2)
- net U3_PC0: now reaches U3.23 (PC0)
- net U3_PC0: now also U3_XT_L1.4 (Pin_4)
- net U3_PC1: now reaches U3.24 (PC1)
- net U3_PC1: now also U3_XT_L1.5 (Pin_5)
- net U3_PC2: now reaches U3.25 (PC2)
- net U3_PC2: now also U3_XT_L1.6 (Pin_6)
- net U3_PC3: now reaches U3.26 (PC3)
- net U3_PC3: now also U3_XT_L1.7 (Pin_7)
- net U3_PC4: now reaches U3.27 (PC4)
- net U3_PC4: now also U3_XT_L1.8 (Pin_8)
- net U3_PD0: now reaches U3.30 (PD0)
- net U3_PD0: now also U3_XT_R1.1 (Pin_1)
- net U3_PD1: now reaches U3.31 (PD1)
- net U3_PD1: now also U3_XT_R1.2 (Pin_2)
- net U3_PD2: now reaches U3.32 (PD2)
- net U3_PD2: now also U3_XT_R1.3 (Pin_3)
- net U3_PB6: now reaches U3.7 (PB6/XTAL1)
- net U3_PB6: now also C3.1, Y_U3.2
- net U3_PB7: now reaches U3.8 (PB7/XTAL2)
- net U3_PB7: now also C4.1, Y_U3.1
- net U3_PD5: now reaches U3.9 (PD5)
- net U3_PD5: now also U3_XT_R1.6 (Pin_6)
- net U4_PD3: now reaches U4.1 (PD3)
- net U4_PD3: now also U4_XT_R1.4 (Pin_4)
- net U4_PD6: now reaches U4.10 (PD6)
- net U4_PD6: now also U4_XT_R1.7 (Pin_7)
- net U4_PD7: now reaches U4.11 (PD7)
- net U4_PD7: now also U4_XT_R1.8 (Pin_8)
- net U4_PB0: now reaches U4.12 (PB0)
- net U4_PB0: now also R29.2
- net U4_PB1: now reaches U4.13 (PB1)
- net U4_PB1: now also U4_XT_L1.3 (Pin_3)
- net U4_ADC6: now reaches U4.19 (ADC6)
- net U4_ADC6: now also U4_XT_L1.1 (Pin_1)
- net U4_PD4: now reaches U4.2 (PD4)
- net U4_PD4: now also U4_XT_R1.5 (Pin_5)
- net U4_ADC7: now reaches U4.22 (ADC7)
- net U4_ADC7: now also U4_XT_L1.2 (Pin_2)
- net U4_PC0: now reaches U4.23 (PC0)
- net U4_PC0: now also U4_XT_L1.4 (Pin_4)
- net U4_PC1: now reaches U4.24 (PC1)
- net U4_PC1: now also U4_XT_L1.5 (Pin_5)
- net U4_PC2: now reaches U4.25 (PC2)
- net U4_PC2: now also U4_XT_L1.6 (Pin_6)
- net U4_PC3: now reaches U4.26 (PC3)
- net U4_PC3: now also U4_XT_L1.7 (Pin_7)
- net U4_PC4: now reaches U4.27 (PC4)
- net U4_PC4: now also U4_XT_L1.8 (Pin_8)
- net U4_PD0: now reaches U4.30 (PD0)
- net U4_PD0: now also U4_XT_R1.1 (Pin_1)
- net U4_PD1: now reaches U4.31 (PD1)
- net U4_PD1: now also U4_XT_R1.2 (Pin_2)
- net U4_PD2: now reaches U4.32 (PD2)
- net U4_PD2: now also U4_XT_R1.3 (Pin_3)
- net U4_PB6: now reaches U4.7 (PB6/XTAL1)
- net U4_PB6: now also C1.1, Y_U4.2
- net U4_PB7: now reaches U4.8 (PB7/XTAL2)
- net U4_PB7: now also C2.1, Y_U4.1
- net U4_PD5: now reaches U4.9 (PD5)
- net U4_PD5: now also U4_XT_R1.6 (Pin_6)
- removed net +5V: J3.2 (VCC), J4.2 (VCC), J5.2 (VCC)
- removed net GND: BZ1.2 (+), J3.6 (GND), J4.6 (GND), J5.6 (GND)
- new net: R29.1, Window_1.2 (A) (x2)
Other:
- company: (none) -> JP TOUTANT, JEREMY DIAPHRASE, MOHAND CHAHED
- title: (none) -> SPI SECTION
- moved on the sheet: BZ1, J11, J12, J3, J4, J5, J_SPI_3, J_SPI_4, J_SPI_5, Q1, Q2, R1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
