File: kicad/untitled.kicad_sch (KiCad schematic)
At the start: 42 parts, among them J11 Conn_01x02_Socket, J12 Conn_01x02_Socket, J3 AVR-ISP-6, J4 AVR-ISP-6, J5 AVR-ISP-6, Q1 NMOS, Q2 NMOS, SW4 SW_SPDT, U3 ATmega8A-A, U3_PW1 Conn_01x03_MountingPin, U3_XT_L1 Conn_01x08, U3_XT_R1 Conn_01x08, U4 ATmega8A-A, U4_PW1 Conn_01x03_MountingPin, U4_XT_L1 Conn_01x08, U4_XT_R1 Conn_01x08, U5 ATmega8A-A, U5_PW1 Conn_01x03_MountingPin, U5_XT1 Conn_01x14

Commit message: switch to SPIs
Parts:
- J3, J4, J5: footprint JPLibrary:SPI_prog -> JP_Library:SPI_prog
Changed lines of the file:
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@@
       (effects (font (size 1.27 1.27)) (justify right) hide)
     )
-    (property "Footprint" "JPLibrary:SPI_prog" (at 278.13 96.52 90)
+    (property "Footprint" "JP_Library:SPI_prog" (at 278.13 96.52 90)
       (effects (font (size 1.27 1.27)) hide)
     )
@@
       (effects (font (size 1.27 1.27)) (justify right))
     )
-    (property "Footprint" "JPLibrary:SPI_prog" (at 96.52 95.25 90)
+    (property "Footprint" "JP_Library:SPI_prog" (at 96.52 95.25 90)
       (effects (font (size 1.27 1.27)) hide)
     )
@@
       (effects (font (size 1.27 1.27)) (justify right) hide)
     )
-    (property "Footprint" "JPLibrary:SPI_prog" (at 184.15 99.06 90)
-      (effects (font (size 1.27 1.27)) hide)
-    )
+    (property "Footprint" "JP_Library:SPI_prog" (at 184.15 99.06 90)
+      (effects (font (size 1.27 1.27)) hide)
+    )
